File: Hardware/USBhub/USBhub.kicad_sch (KiCad schematic)
At the start: 6 parts

Commit message: small updates
Parts:
- added D1, D2, D3, D4, D5, D6, D7: LED, LED_SMD:LED_PLCC-2, symbol Device:LED
- added H1, H10, H2, H3, H4, H5, H6, H7, H8, H9: MountingHole, MountingHole:MountingHole_2.7mm_M2.5, symbol Mechanical:MountingHole
- added J4: USB_A, Connector_USB:USB_A_Wuerth_614004134726_Horizontal, symbol Connector:USB_A
- added SW1, SW3: SW_Push, symbol Switch:SW_Push
- added SW2: SW_SPDT_MSM, symbol Switch:SW_SPDT_MSM
- added U3, U4: NUP4202, Package_TO_SOT_SMD:SOT-363_SC-70-6, symbol Power_Protection:NUP4202
- added U5, U6: MIC2097-1YMT, symbol MyLib:MIC2097-1YMT
- J3: renamed from J?; footprint (none) -> Connector_USB:USB_A_Wuerth_614004134726_Horizontal
- gave numbers to parts that had none: 5
Connections:
- net at U2.30 (USBDM_UP): now also J1.2 (D-), U1.6
- net at U2.31 (USBDP_UP): now also J1.3 (D+), U1.4
Other:
- note added: "Settings for USB hub: * * *"
- moved on the sheet: J3, Y1
